File: RAILBooster-Shield/board/Railbooster Shield.brd (EAGLE design)
At the start: 68.6 x 53.3 mm, 39 parts, among them IC1 LMD18200, IC2 LM358D, IC3 V_REG_LD1085D2, IC4 IC_555-SOIC8, J1 POWER_JACKPTH, U1 ARDUINOR3-DIMENSION, X4 SCREWTERMINAL-5.08-2

Commit message: Update to remove rouge connector
Parts:
- removed JP1: M02SPRING-2.54-RA, SparkFun-Connectors:SPRINGTERMINAL-2.54MM-2
Changed lines of the file:
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@@
 <attribute name="NAME" x="30.582" y="12.3" size="1.27" layer="25" align="bottom-center"/>
 </element>
-<element name="JP1" library="SparkFun-Connectors" package="SPRINGTERMINAL-2.54MM-2" value="M02SPRING-2.54-RA" x="64" y="43.5" rot="R90"/>
 </elements>
 <signals>
